File: Arm/A/Arm.kicad_pcb (KiCad board)
At the start: 2 copper layers, 87.7 x 254.8 mm, 62 parts, among them J1 Conn_01x04, J2 Conn_01x04, U1 SM351LT, U2 SM351LT

Commit message: adapt length to fit 26" wheels
Parts:
- REF**: value bicycle -> bicycle-silkscreen-5x6mm; footprint Library:bicycle -> Library:bicycle-silkscreen-5x6mm
- moved FID3 34.7 mm to (99.9, 48.6)
- moved H1 34.7 mm to (102.0, 50.7)
- moved H17 34.7 mm to (116.0, 50.7)
- moved D32 34.1 mm to (109.0, 50.1)
- moved D31 33.0 mm to (109.0, 57.0)
- moved D30 31.9 mm to (109.0, 63.9)
- moved D29 30.8 mm to (109.0, 70.8)
- moved D28 29.7 mm to (109.0, 77.7)
- moved D27 28.6 mm to (109.0, 84.6)
- moved D26 27.5 mm to (109.0, 91.5)
- moved D25 26.4 mm to (109.0, 98.4)
- moved U1 26.0 mm to (102.1, 62.1)
- moved D24 25.3 mm to (109.0, 105.3)
- moved D23 24.2 mm to (109.0, 112.2)
- moved D22 23.1 mm to (109.0, 119.1)
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Routing:
- net /HAL_SENSOR: track 272.9 -> 247.3 mm
- net GND: track 47.1 -> 54.3 mm
- net Net-(D7-DOUT): track 8.72 -> 6.81 mm
- net Net-(D5-DOUT): track 8.72 -> 6.81 mm
- net Net-(D15-DOUT): track 8.72 -> 6.81 mm
- net /DOUT_16: track 8.72 -> 6.81 mm
- net Net-(D26-DOUT): track 8.72 -> 6.81 mm
- net Net-(D29-DOUT): track 8.72 -> 6.81 mm
- net /DOUT_8: track 8.72 -> 6.81 mm
- net Net-(D6-DOUT): track 8.72 -> 6.81 mm
- net Net-(D17-DOUT): track 8.72 -> 6.81 mm
- net Net-(D12-DOUT): track 8.72 -> 6.81 mm
- net Net-(D11-DOUT): track 8.72 -> 6.81 mm
- net Net-(D4-DOUT): track 8.72 -> 6.81 mm
- net Net-(D25-DOUT): track 8.72 -> 6.81 mm
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Other:
- board size 87.7 x 254.8 mm -> 87.7 x 220.1 mm
- board text added: "Max for 26{dblquote}"
- board text added: "Rev 1.0"
- board text added: "SpokeSpice26"
- board text removed: "Rev A"
- board text removed: "SpokeSpice"
